File: hardware/thermocouple.kicad_pcb (KiCad board)
At the start: 2 copper layers, 40 x 30 mm, 26 parts, among them J101 AKL_5_2, P101 CON-SENSOR, U101 M24C64, U102 MAX31856, U103 DRILL, U104 DRILL, U105 DRILL, U106 DRILL

Commit message: rename thermocouple connector
Parts:
- J101: value AKL_5_2 -> THERM
Changed lines of the file:
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@@
-(kicad_pcb (version 4) (host pcbnew "(2015-03-18 BZR 5525)-product")
+(kicad_pcb (version 4) (host pcbnew 4.0.2+e4-6225~38~ubuntu15.10.1-stable)
   (general
     (links 42)
     (no_connects 0)
-    (area 149.934499 124.734499 190.315501 155.115501)
+    (area 149.219339 124.019339 282.371482 165.089523)
     (thickness 1.6002)
     (drawings 12)
@@
       (effects (font (size 1 1) (thickness 0.15)))
     )
-    (fp_text value AKL_5_2 (at 0 -0.5 270) (layer F.Fab)
+    (fp_text value THERM (at 0 -0.5 270) (layer F.Fab)
       (effects (font (size 1 1) (thickness 0.15)))
     )
