File: hardware/thermocouple.kicad_pcb (KiCad board)
At the start: 2 copper layers, 40 x 30 mm, 26 parts, among them J101 THERM, P101 CON-SENSOR, U101 M24C64, U102 MAX31856, U103 DRILL, U104 DRILL, U105 DRILL, U106 DRILL

Commit message: change capacitor value
Parts:
- C105: value 10nF -> 100nF
Changed lines of the file:
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@@
-(kicad_pcb (version 4) (host pcbnew 4.0.2+e4-6225~38~ubuntu15.10.1-stable)
+(kicad_pcb (version 4) (host pcbnew 4.0.7-e2-6376~58~ubuntu17.04.1)
   (general
     (links 42)
     (no_connects 0)
-    (area 149.219339 124.019339 282.371482 165.089523)
+    (area 149.219339 124.019339 282.27147 165.489573)
     (thickness 1.6002)
     (drawings 12)
@@
       (effects (font (size 0.2 0.2) (thickness 0.05)))
     )
-    (fp_text value 10nF (at 0.05 -0.375 270) (layer F.SilkS)
-      (effects (font (size 0.2 0.2) (thickness 0.05)))
-    )
+    (fp_text value 100nF (at 0.05 -0.375 270) (layer F.SilkS)
+      (effects (font (size 0.2 0.2) (thickness 0.05)))
+    )
